File: schematics/src/voiceboard/voiceboard.brd (EAGLE design)
At the start: 50.8 x 99.1 mm, 53 parts, among them IC1 LM13700N, IC2 TL074P, IC3 TL072P, Q1 BC557C, Q2 BC557C

Commit message: Added Status & Images
Routing:
- net N$13: track 66.7 -> 68.3 mm
- net +12V: vias 3 -> 2
Changed lines of the file:
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@@
 <wire x1="29.21" y1="23.495" x2="27.94" y2="22.225" width="0.6096" layer="1"/>
 <wire x1="26.67" y1="42.545" x2="20.32" y2="42.545" width="0.6096" layer="16"/>
-<wire x1="12.7" y1="32.385" x2="17.145" y2="32.385" width="0.6096" layer="16"/>
-<wire x1="17.145" y1="32.385" x2="18.415" y2="31.115" width="0.6096" layer="16"/>
-<wire x1="18.415" y1="31.115" x2="29.21" y2="31.115" width="0.6096" layer="16"/>
-<via x="29.21" y="31.115" extent="1-16" drill="0.35"/>
+<wire x1="12.7" y1="32.385" x2="17.145" y2="32.385" width="0.6096" layer="1"/>
+<wire x1="17.145" y1="32.385" x2="18.415" y2="31.115" width="0.6096" layer="1"/>
+<wire x1="18.415" y1="31.115" x2="29.21" y2="31.115" width="0.6096" layer="1"/>
 </signal>
 <signal name="N$2">
@@
 <wire x1="37.465" y1="70.485" x2="40.64" y2="73.66" width="0.4064" layer="16"/>
 <wire x1="40.64" y1="73.66" x2="41.91" y2="73.66" width="0.4064" layer="16"/>
-<wire x1="12.7" y1="29.845" x2="15.875" y2="29.845" width="0.4064" layer="1"/>
-<wire x1="15.875" y1="29.845" x2="18.415" y2="32.385" width="0.4064" layer="1"/>
-<wire x1="18.415" y1="32.385" x2="18.415" y2="47.625" width="0.4064" layer="1"/>
+<wire x1="12.7" y1="29.845" x2="12.065" y2="29.845" width="0.4064" layer="1"/>
+<wire x1="12.065" y1="29.845" x2="10.795" y2="31.115" width="0.4064" layer="1"/>
+<wire x1="10.795" y1="31.115" x2="10.795" y2="32.385" width="0.4064" layer="1"/>
+<wire x1="10.795" y1="32.385" x2="12.065" y2="33.655" width="0.4064" layer="1"/>
+<wire x1="12.065" y1="33.655" x2="14.605" y2="33.655" width="0.4064" layer="1"/>
+<wire x1="14.605" y1="33.655" x2="18.415" y2="37.465" width="0.4064" layer="1"/>
+<wire x1="18.415" y1="37.465" x2="18.415" y2="47.625" width="0.4064" layer="1"/>
 <wire x1="18.415" y1="47.625" x2="23.495" y2="52.705" width="0.4064" layer="1"/>
 <via x="23.495" y="70.485" extent="1-16" drill="0.35"/>
